File: ORANGE_HAT/design/ORANGE_PI_4_PRO/ORANGE_PI_4_PRO.kicad_sch (KiCad schematic)
At the start: 2 parts, among them P1 Conn_02x20_Odd_Even, P2 Conn_02x20_Odd_Even

Commit message: VIAS
Parts:
- added P3: Conn_02x20_Odd_Even, Connector_PinSocket_2.54mm:PinSocket_2x20_P2.54mm_Vertical, symbol Connector_Generic:Conn_02x20_Odd_Even
Connections:
- net +3.3V: now also P3.33 (Pin_33), P3.34 (Pin_34)
- net +5V: now also P3.35 (Pin_35), P3.36 (Pin_36)
- net GND: now also P3.17 (Pin_17), P3.18 (Pin_18), P3.19 (Pin_19), P3.20 (Pin_20), P3.37 (Pin_37), P3.38 (Pin_38), P3.39 (Pin_39), P3.40 (Pin_40)
- net PB2: now also P3.1 (Pin_1)
- net PB3: now also P3.3 (Pin_3)
- net PB4: now also P3.5 (Pin_5)
- net PB5: now also P3.7 (Pin_7)
- net PD0: now also P3.2 (Pin_2)
- net PD1: now also P3.4 (Pin_4)
- net PD2: now also P3.6 (Pin_6)
- net PD23: now also P3.24 (Pin_24)
- net PD3: now also P3.8 (Pin_8)
- net PD4: now also P3.10 (Pin_10)
- net PD5: now also P3.12 (Pin_12)
- net PD6: now also P3.14 (Pin_14)
- net PD7: now also P3.16 (Pin_16)
- net PE1: now also P3.29 (Pin_29)
- net PE12: now also P3.22 (Pin_22)
- net PE2: now also P3.31 (Pin_31)
- net PE3: now also P3.30 (Pin_30)
- net PE4: now also P3.32 (Pin_32)
- net PK24: now also P3.26 (Pin_26)
- net PK25: now also P3.28 (Pin_28)
- net PL12: now also P3.25 (Pin_25)
- net PL13: now also P3.27 (Pin_27)
- net PL4: now also P3.9 (Pin_9)
- net PL5: now also P3.11 (Pin_11)
- net PL6: now also P3.13 (Pin_13)
- net PL7: now also P3.15 (Pin_15)
- net PL8: now also P3.21 (Pin_21)
- net PL9: now also P3.23 (Pin_23)
Other:
- note added: "BIAS"
